Commit message: rtk因子加入优化

File: launch/include/config/robot.urdf.xacro (robot description, xacro)
@@ -27,3 +27,9 @@
     <origin xyz="0 0 0" rpy="0 0 0" />
   </joint>
+  <link name="livox_frame"> </link>
+  <joint name="livox_frame_joint" type="fixed">
+    <parent link="chassis_link" />
+    <child link="livox_frame" />
+    <origin xyz="0 0 0" rpy="0 0 0" />
+  </joint>
 </robot>
